File: Digital Lockin PRE Autorouter.brd (EAGLE design)
At the start: 76.2 x 94.9 mm, 24 parts, among them IC1 OPA2650E, IC2 LM358D, T2 NPN, U2 RASPBERRY_PICOSMD-TH, U5 TL431AIDBZR

Commit message: Final with Overlap
Routing:
- net GND: track 382.2 -> 0.00 mm, vias 12 -> 4
- net 5V: track 154.4 -> 0.00 mm, vias 3 -> 0
- net ADCMID: track 127.4 -> 0.00 mm, vias 2 -> 0
- net AMPOUT: track 79.4 -> 0.00 mm
- net LEDCTRL: track 67.4 -> 0.00 mm
- net 3V3: track 60.0 -> 0.00 mm
- net ADCREF: track 55.8 -> 0.00 mm
- net N$6: track 50.2 -> 0.00 mm
- net N$1: track 28.2 -> 0.00 mm
- net N$13: track 27.4 -> 0.00 mm
- net N$5: track 25.4 -> 0.00 mm
- net N$2: track 20.1 -> 0.00 mm
- net N$9: track 16.6 -> 0.00 mm
- net N$10: track 11.3 -> 0.00 mm
- net N$20: track 7.35 -> 0.00 mm
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- removed copper zone on layer 1, net GND
- removed copper zone on layer 16, net GND
